File: pcb/ble.kicad_pcb (KiCad board)
At the start: 2 copper layers, 23.7 x 14.5 mm, 14 parts, among them J1 Conn_01x05, J2 Conn_01x09, J3 Conn_01x06, J5 Conn_01x01, J6 Conn_01x01, SW1 SW_Push, U1 BME280

Commit message: Add github note
Other:
- board text added: "github.com/NerdyProjects/ble-thermometer"
Changed lines of the file:
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@@
     (area 105.299999 107.399999 129.200001 122.100001)
     (thickness 1.6)
-    (drawings 25)
+    (drawings 26)
     (tracks 113)
     (zones 0)
@@
     )
   )
+  (gr_text github.com/NerdyProjects/ble-thermometer (at 116.5 108) (layer F.SilkS)
+    (effects (font (size 0.5 0.5) (thickness 0.1)))
+  )
   (gr_text "Matthias Larisch" (at 123.1 121) (layer F.SilkS)

Commit message: Add pcb image
Routing:
- net GND: track 48.6 -> 52.8 mm, vias 3 -> 9
- net SDA: track 37.9 -> 41.4 mm, vias 0 -> 1
- net SCL: track 38.9 -> 42.3 mm, vias 0 -> 1
- added copper zone on F.Cu, net GND
Other:
- rule pad_to_mask_clearance: 0.2 -> 0.05
- board text removed: "CR1632 COIN CELL"
